Commit message: preJan28

File: mir/mir_description/urdf/include/common.gazebo.xacro (robot description, xacro)
@@ -2,5 +2,5 @@
 <robot xmlns:xacro="http://ros.org/wiki/xacro">
   <xacro:macro name="controller_plugin_gazebo" params="robot_namespace">
-    <gazebo>
+    <!-- <gazebo>
       <plugin name="gazebo_ros_control" filename="libgazebo_ros_control.so">
         <xacro:unless value="${robot_namespace == ''}">
@@ -10,5 +10,5 @@
         <legacyModeNS>false</legacyModeNS>
       </plugin>
-    </gazebo>
+    </gazebo> -->
   </xacro:macro>
 </robot>

File: mir/mir_description/urdf/include/imu.gazebo.urdf.xacro (robot description, xacro)
@@ -12,16 +12,10 @@
   <xacro:macro name="imu_gazebo" params="link imu_topic update_rate">
     <gazebo>
-      <plugin name="imu_plugin" filename="libhector_gazebo_ros_imu.so">
-        <updateRate>${update_rate}</updateRate>
-        <bodyName>${link}</bodyName>
-        <frameId>${imu_frame}</frameId>  <!-- from real MiR -->
-        <topicName>${imu_topic}</topicName>
-        <accelDrift>0.0 0.0 0.0</accelDrift>
-        <accelGaussianNoise>${sqrt(5e-05)} ${sqrt(0.0001)} ${sqrt(0.00013)}</accelGaussianNoise>    <!-- real MiR linear_acceleration_covariance [5e-05, 0.0, 0.0, 0.0, 0.0001, 0.0, 0.0, 0.0, 0.00013] -->
-        <rateDrift>0.0 0.0 0.0</rateDrift>
-        <rateGaussianNoise>${sqrt(8e-06)} ${sqrt(8e-06)} ${sqrt(3e-07)}</rateGaussianNoise>         <!-- real MiR angular_velocity_covariance [8e-06, 0.0, 0.0, 0.0, 8e-06, 0.0, 0.0, 0.0, 3e-07] -->
-        <yawDrift>0.0</yawDrift>
-        <yawGaussianNoise>${sqrt(0.1)}</yawGaussianNoise>                                           <!-- real MiR orientation_covariance [0.1, 0.0, 0.0, 0.0, 0.1, 0.0, 0.0, 0.0, 0.1] -->
-      </plugin>
+      <sensor name="imu_sensor" type="imu">
+          <always_on>1</always_on>
+          <update_rate>${update_rate}</update_rate>
+          <visualize>true</visualize>
+          <topic>${imu_topic}</topic>
+      </sensor>
     </gazebo>
   </xacro:macro>

File: mir/mir_description/urdf/include/mir.gazebo.xacro (robot description, xacro)
@@ -3,5 +3,16 @@
   <xacro:macro name="diff_controller_plugin_gazebo" params="prefix left_wheel_joint right_wheel_joint wheel_separation wheel_radius">
     <gazebo>
-      <plugin name="diff_drive_controller" filename="libgazebo_ros_diff_drive.so">
+      <!--diff drive plugin-->
+      <plugin
+          filename="gz-sim-diff-drive-system"
+          name="gz::sim::systems::DiffDrive">
+          <left_joint>${left_wheel_joint}</left_joint>
+          <right_joint>${right_wheel_joint}</right_joint>
+          <wheel_separation>${wheel_separation}</wheel_separation>
+          <wheel_radius>${wheel_radius}</wheel_radius>
+          <odom_publish_frequency>1</odom_publish_frequency>
+          <topic>mobile_base_controller/cmd_vel</topic>
+      </plugin>
+      <!-- <plugin name="diff_drive_controller" filename="libgazebo_ros_diff_drive.so">
         <legacyMode>false</legacyMode>
         <alwaysOn>true</alwaysOn>
@@ -22,5 +33,5 @@
         <odometrySource>world</odometrySource>
         <rosDebugLevel>Debug</rosDebugLevel>
-      </plugin>
+      </plugin> -->
     </gazebo>
   </xacro:macro>
@@ -43,5 +54,5 @@
   </xacro:macro>
   <xacro:macro name="p3d_base_controller" params="prefix">
-    <gazebo>
+    <!-- <gazebo>
       <plugin name="p3d_base_controller" filename="libgazebo_ros_p3d.so">
         <alwaysOn>true</alwaysOn>
@@ -54,5 +65,5 @@
         <rpyOffsets>0 0 0</rpyOffsets>
       </plugin>
-    </gazebo>
+    </gazebo> -->
   </xacro:macro>
 </robot>

File: mir/mir_description/urdf/include/mir_v2.urdf.xacro (robot description, xacro)
@@ -204,6 +204,7 @@
       <origin xyz="0.0 0.0 0.25" rpy="0 0 0" />  <!-- same as real MiR -->
     </joint>
-    <link name="${prefix}imu_link" />
-    <xacro:imu_gazebo link="${prefix}imu_link" imu_topic="imu_data" update_rate="50.0" />
+    <link name="${prefix}imu_link">
+      <xacro:imu_gazebo link="${prefix}imu_link" imu_topic="imu_data" update_rate="50.0" />
+    </link>
     <!-- Create an alias for imu_link. This is necessary because the real MiR's
          TF has imu_link, but the imu_data topic is published in the imu_frame

File: mir/mir_description/urdf/include/sick_s300.urdf.xacro (robot description, xacro)
@@ -27,37 +27,31 @@
     </link>
     <gazebo reference="${prefix}${link}">
-      <!-- <material value="Gazebo/Yellow" /> -->
-      <!-- <material value="Gazebo/FlatBlack" /> -->
-      <sensor type="ray" name="${prefix}${link}">
-        <pose>0 0 0 0 0 0</pose>
-        <visualize>false</visualize>
-        <update_rate>12.5</update_rate>
-        <ray>
-          <scan>
-            <horizontal>
-              <samples>541</samples>
-              <resolution>1</resolution>  <!-- has to be 1; actual resolution will be computed from number of samples + min_angle/max_angle -->
-              <min_angle>-2.35619449615</min_angle>
-              <max_angle>2.35619449615</max_angle>
-            </horizontal>
-          </scan>
-          <range>
-            <min>0.05</min>
-            <max>29.0</max>
-            <resolution>0.01</resolution>
-          </range>
-          <noise>
-            <type>gaussian</type>
-            <!-- Noise parameters based on published spec for S300 achieving
-                 "+-29mm" accuracy at range < 3m (~0.01 of the range) at
-                 1 sigma. -->
-            <mean>0.0</mean>
-            <stddev>0.01</stddev>
-          </noise>
-        </ray>
-        <plugin name="gazebo_ros_${link}_controller" filename="libgazebo_ros_laser.so">
-          <frameName>${prefix}${link}</frameName>
-          <topicName>${topic}</topicName>
-        </plugin>
+      <sensor name='${prefix}${link}' type='ray'>
+          <pose relative_to='${prefix}${link}'>0 0 0 0 0 0</pose>
+          <topic>${topic}</topic>
+          <update_rate>12.5</update_rate>
+          <ray>
+              <scan>
+                  <horizontal>
+                      <samples>541</samples>
+                      <resolution>1</resolution>
+                      <min_angle>-2.35619449615</min_angle>
+                      <max_angle>2.35619449615</max_angle>
+                  </horizontal>
+                  <vertical>
+                      <samples>1</samples>
+                      <resolution>0.01</resolution>
+                      <min_angle>0</min_angle>
+                      <max_angle>0</max_angle>
+                  </vertical>
+              </scan>
+              <range>
+                  <min>0.05</min>
+                  <max>29.0</max>
+                  <resolution>0.01</resolution>
+              </range>
+          </ray>
+          <always_on>1</always_on>
+          <visualize>true</visualize>
       </sensor>
     </gazebo>

Commit message: added ros bridge, sensors still not working

File: mir/mir_description/urdf/include/common.gazebo.xacro (robot description, xacro)
@@ -1,4 +1,10 @@
 <?xml version="1.0"?>
 <robot xmlns:xacro="http://ros.org/wiki/xacro">
+  <plugin filename="gz-sim-joint-state-publisher-system"
+    name="gz::sim::systems::JointStatePublisher">
+    <topic>joint_states</topic> <!--from <ros><remapping> -->
+    <joint_name>wheel_left_joint</joint_name>
+    <joint_name>wheel_right_joint</joint_name>
+  </plugin>
   <xacro:macro name="controller_plugin_gazebo" params="robot_namespace">
     <!-- <gazebo>

File: mir/mir_description/urdf/include/imu.gazebo.urdf.xacro (robot description, xacro)
@@ -12,9 +12,22 @@
   <xacro:macro name="imu_gazebo" params="link imu_topic update_rate">
     <gazebo>
-      <sensor name="imu_sensor" type="imu">
-          <always_on>1</always_on>
-          <update_rate>${update_rate}</update_rate>
-          <visualize>true</visualize>
-          <topic>${imu_topic}</topic>
+      <sensor name="tb3_imu" type="imu">
+        <always_on>true</always_on>
+        <update_rate>200</update_rate>
+        <topic>imu</topic>
+        <imu>
+          ... <!-- all the content of <imu> -->
+        </imu>
+      </sensor>
+      <sensor name="camera" type="camera">
+        <always_on>true</always_on>
+        <visualize>true</visualize>
+        <update_rate>30</update_rate>
+        <topic>camera/image_raw</topic>
+        <gz_frame_id>camera_rgb_frame</gz_frame_id>
+        <camera name="intel_realsense_r200">
+          <camera_info_topic>camera/camera_info</camera_info_topic>
+          ... <!-- all the content of <camera> from the original -->
+        </camera>
       </sensor>
     </gazebo>

File: mir/mir_description/urdf/include/mir.gazebo.xacro (robot description, xacro)
@@ -1,16 +1,23 @@
 <?xml version="1.0"?>
 <robot xmlns:xacro="http://ros.org/wiki/xacro">
-  <xacro:macro name="diff_controller_plugin_gazebo" params="prefix left_wheel_joint right_wheel_joint wheel_separation wheel_radius">
+  <xacro:macro name="diff_controller_plugin_gazebo" params="prefix controller_config_file">
+    <!-- <xacro:gazebo.controller config_file="${controller_config_file}" namespace="${prefix}" /> -->
     <gazebo>
-      <!--diff drive plugin-->
-      <plugin
-          filename="gz-sim-diff-drive-system"
-          name="gz::sim::systems::DiffDrive">
-          <left_joint>${left_wheel_joint}</left_joint>
-          <right_joint>${right_wheel_joint}</right_joint>
-          <wheel_separation>${wheel_separation}</wheel_separation>
-          <wheel_radius>${wheel_radius}</wheel_radius>
-          <odom_publish_frequency>1</odom_publish_frequency>
-          <topic>mobile_base_controller/cmd_vel</topic>
+      <plugin filename="gz-sim-diff-drive-system" name="gz::sim::systems::DiffDrive">
+        <!-- Remove <ros> tag. -->
+        <!-- wheels -->
+        <left_joint>wheel_left_joint</left_joint>
+        <right_joint>wheel_right_joint</right_joint>
+        <!-- kinematics -->
+        <wheel_separation>0.287</wheel_separation>
+        <wheel_radius>0.033</wheel_radius> <!-- computed from <wheel_diameter> in the original plugin-->
+        <!-- limits -->
+        <max_linear_acceleration>0.033</max_linear_acceleration> <!-- computed from <max_linear_acceleration> in the original plugin-->
+        <topic>cmd_vel</topic> <!-- from <commant_topic> -->
+        <odom_topic>odom</odom_topic> <!-- from <odometry_topic> -->
+        <frame_id>odom</frame_id> <!-- from <odometry_frame> -->
+        <child_frame_id>base_footprint</child_frame_id> <!-- from <robot_base_frame> -->
+        <odom_publisher_frequency>30</odom_publisher_frequency> <!-- from <update_rate>-->
+        <tf_topic>/tf</tf_topic> <!-- Short topic name for tf output -->
       </plugin>
       <!-- <plugin name="diff_drive_controller" filename="libgazebo_ros_diff_drive.so">

File: mir/mir_description/urdf/include/mir_v2.urdf.xacro (robot description, xacro)
@@ -174,5 +174,5 @@
     </link>
   </xacro:macro>
-  <xacro:macro name="mir" params="prefix">
+  <xacro:macro name="mir" params="prefix controller_config_file">
     <link name="${prefix}base_footprint" />
     <joint name="${prefix}base_joint" type="fixed">
@@ -259,5 +259,6 @@
     <!-- set the gazebo friction parameters for the wheels -->
     <xacro:set_all_wheel_frictions prefix="${prefix}"/>
-    <xacro:p3d_base_controller prefix="${prefix}" />
+    <!-- <xacro:diff_controller_plugin_gazebo prefix="${prefix}" controller_config_file="${controller_config_file}" /> -->
+    <!-- <xacro:p3d_base_controller prefix="${prefix}" /> -->
   </xacro:macro>
 </robot>

File: mir/mir_description/urdf/include/sick_s300.urdf.xacro (robot description, xacro)
@@ -27,9 +27,10 @@
     </link>
     <gazebo reference="${prefix}${link}">
-      <sensor name='${prefix}${link}' type='ray'>
+      <sensor name='${prefix}${link}' type='gpu_lidar'>
           <pose relative_to='${prefix}${link}'>0 0 0 0 0 0</pose>
           <topic>${topic}</topic>
           <update_rate>12.5</update_rate>
-          <ray>
+          <gz_frame_id>base_scan</gz_frame_id>
+          <lidar>
               <scan>
                   <horizontal>
@@ -51,6 +52,6 @@
                   <resolution>0.01</resolution>
               </range>
-          </ray>
-          <always_on>1</always_on>
+          </lidar>
+          <always_on>true</always_on>
           <visualize>true</visualize>
       </sensor>

File: mir/mir_description/urdf/mir.urdf.xacro (robot description, xacro)
@@ -2,4 +2,5 @@
 <robot xmlns:xacro="http://ros.org/wiki/xacro"
        name="mir" >
+  <xacro:arg name="controller_config_file" default="$(find mir_description)/config/diff_drive_controller.yaml" />
   <!-- MiR base -->
   <xacro:include filename="$(find mir_description)/urdf/include/mir_v2.urdf.xacro" />
@@ -13,5 +14,6 @@
     <xacro:property name="prefix" value="${tf_prefix_}/" />
   </xacro:unless>
-  <xacro:mir prefix="${prefix}" />
+  <xacro:mir prefix="${prefix}" controller_config_file="$(arg controller_config_file)"/>
+  <xacro:arg name="simulation_engine" default="ignition-gazebo" />
   <xacro:controller_plugin_gazebo robot_namespace=""/>
   <!-- instead of the controller_plugin_gazebo, you can use the diffdrive controller like this
