Commit message: added diff drive gz

File: mir/mir_description/urdf/include/common.gazebo.xacro (robot description, xacro)
@@ -1,20 +1,145 @@
 <?xml version="1.0"?>
 <robot xmlns:xacro="http://ros.org/wiki/xacro">
-  <plugin filename="gz-sim-joint-state-publisher-system"
-    name="gz::sim::systems::JointStatePublisher">
-    <topic>joint_states</topic> <!--from <ros><remapping> -->
-    <joint_name>wheel_left_joint</joint_name>
-    <joint_name>wheel_right_joint</joint_name>
-  </plugin>
-  <xacro:macro name="controller_plugin_gazebo" params="robot_namespace">
-    <!-- <gazebo>
-      <plugin name="gazebo_ros_control" filename="libgazebo_ros_control.so">
-        <xacro:unless value="${robot_namespace == ''}">
-          <robotNamespace>${robot_namespace}</robotNamespace>
-        </xacro:unless>
-        <controlPeriod>0.001</controlPeriod>
-        <legacyModeNS>false</legacyModeNS>
+  <xacro:include filename="$(find mir_description)/urdf/include/mir.gazebo.xacro" />
+  <xacro:macro name="caster_wheels_add_gazebo" params="prefix location">
+      <joint name="${prefix}${location}_caster_wheel_joint">
+        <state_interface name="position"/>
+        <state_interface name="velocity"/>
+      </joint>
+      <joint name="${prefix}${location}_caster_rotation_joint">
+        <state_interface name="position"/>
+        <state_interface name="velocity"/>
+      </joint>
+  </xacro:macro>
+  <xacro:macro name="gz_ros2" params="prefix">
+    <ros2_control name="GazeboSimSystem" type="system">
+      <hardware>
+        <plugin>gz_ros2_control/GazeboSimSystem</plugin>
+      </hardware>
+      <joint name="${prefix}left_wheel_joint">
+        <command_interface name="velocity">
+          <param name="min">-1</param>
+          <param name="max">1</param>
+        </command_interface>
+        <state_interface name="position"/>
+        <state_interface name="velocity"/>
+        <state_interface name="effort"/>
+      </joint>
+      <joint name="${prefix}right_wheel_joint">
+        <command_interface name="velocity">
+          <param name="min">-1</param>
+          <param name="max">1</param>
+        </command_interface>
+        <state_interface name="position"/>
+        <state_interface name="velocity"/>
+        <state_interface name="effort"/>
+      </joint>
+      <xacro:caster_wheels_add_gazebo prefix="${prefix}" location="bl" />
+      <xacro:caster_wheels_add_gazebo prefix="${prefix}" location="fr" />
+      <xacro:caster_wheels_add_gazebo prefix="${prefix}" location="br" />
+      <xacro:caster_wheels_add_gazebo prefix="${prefix}" location="fl" />
+    </ros2_control>
+    <gazebo>
+      <!-- Joint state publisher -->
+      <plugin filename="gz_ros2_control-system" name="gz_ros2_control::GazeboSimROS2ControlPlugin">
+        <parameters>$(find mir_description)/config/diff_drive_controller_velocity.yaml</parameters>
+        <controller_manager_name>mir_controller_manager</controller_manager_name>
+        <ros>
+          <namespace></namespace>
+          <remapping>/robot_description:=/robot_description</remapping>
+        </ros>
       </plugin>
-    </gazebo> -->
+      <plugin
+        filename="gz-sim-sensors-system" name="gz::sim::systems::Sensors">
+        <render_engine>ogre2</render_engine>
+      </plugin>
+      <plugin
+        filename="gz-sim-imu-system"
+        name="gz::sim::systems::Imu">
+      </plugin>
+    </gazebo>
+    <!-- IMU  -->
+    <gazebo reference="imu_link">
+      <sensor name="imu_sensor" type="imu">
+        <always_on>1</always_on>
+        <update_rate>41</update_rate>
+        <visualize>true</visualize>
+        <topic>imu</topic>
+        <imu>
+          <enable_orientation>0</enable_orientation>
+          <angular_velocity>
+            <x>
+              <noise type="gaussian">
+                <mean>0</mean>
+                <stddev>0.009</stddev>
+                <bias_mean>0.00075</bias_mean>
+                <bias_stddev>0.005</bias_stddev>
+                <dynamic_bias_stddev>0.00002</dynamic_bias_stddev>
+                <dynamic_bias_correlation_time>400.0</dynamic_bias_correlation_time>
+                <precision>0.00025</precision>
+              </noise>
+            </x>
+            <y>
+              <noise type="gaussian">
+                <mean>0</mean>
+                <stddev>0.009</stddev>
+                <bias_mean>0.00075</bias_mean>
+                <bias_stddev>0.005</bias_stddev>
+                <dynamic_bias_stddev>0.00002</dynamic_bias_stddev>
+                <dynamic_bias_correlation_time>400.0</dynamic_bias_correlation_time>
+                <precision>0.00025</precision>
+              </noise>
+            </y>
+            <z>
+              <noise type="gaussian">
+                <mean>0</mean>
+                <stddev>0.009</stddev>
+                <bias_mean>0.00075</bias_mean>
+                <bias_stddev>0.005</bias_stddev>
+                <dynamic_bias_stddev>0.00002</dynamic_bias_stddev>
+                <dynamic_bias_correlation_time>400.0</dynamic_bias_correlation_time>
+                <precision>0.00025</precision>
+              </noise>
+            </z>
+          </angular_velocity>
+          <linear_acceleration>
+            <x>
+              <noise type="gaussian">
+                <mean>0</mean>
+                <stddev>0.021</stddev>
+                <bias_mean>0.05</bias_mean>
+                <bias_stddev>0.0075</bias_stddev>
+                <dynamic_bias_stddev>0.000375</dynamic_bias_stddev>
+                <dynamic_bias_correlation_time>175.0</dynamic_bias_correlation_time>
+                <precision>0.005</precision>
+              </noise>
+            </x>
+            <y>
+              <noise type="gaussian">
+                <mean>0</mean>
+                <stddev>0.021</stddev>
+                <bias_mean>0.05</bias_mean>
+                <bias_stddev>0.0075</bias_stddev>
+                <dynamic_bias_stddev>0.000375</dynamic_bias_stddev>
+                <dynamic_bias_correlation_time>175.0</dynamic_bias_correlation_time>
+                <precision>0.005</precision>
+              </noise>
+            </y>
+            <z>
+              <noise type="gaussian">
+                <mean>0</mean>
+                <stddev>0.021</stddev>
+                <bias_mean>0.05</bias_mean>
+                <bias_stddev>0.0075</bias_stddev>
+                <dynamic_bias_stddev>0.000375</dynamic_bias_stddev>
+                <dynamic_bias_correlation_time>175.0</dynamic_bias_correlation_time>
+                <precision>0.005</precision>
+              </noise>
+            </z>
+          </linear_acceleration>
+        </imu>
+      </sensor>
+    </gazebo>
+    <xacro:set_all_wheel_frictions prefix="${prefix}" />
   </xacro:macro>
 </robot>

File: mir/mir_description/urdf/include/mir.gazebo.xacro (robot description, xacro)
@@ -1,46 +1,4 @@
 <?xml version="1.0"?>
 <robot xmlns:xacro="http://ros.org/wiki/xacro">
-  <xacro:macro name="diff_controller_plugin_gazebo" params="prefix controller_config_file">
-    <!-- <xacro:gazebo.controller config_file="${controller_config_file}" namespace="${prefix}" /> -->
-    <gazebo>
-      <plugin filename="gz-sim-diff-drive-system" name="gz::sim::systems::DiffDrive">
-        <!-- Remove <ros> tag. -->
-        <!-- wheels -->
-        <left_joint>wheel_left_joint</left_joint>
-        <right_joint>wheel_right_joint</right_joint>
-        <!-- kinematics -->
-        <wheel_separation>0.287</wheel_separation>
-        <wheel_radius>0.033</wheel_radius> <!-- computed from <wheel_diameter> in the original plugin-->
-        <!-- limits -->
-        <max_linear_acceleration>0.033</max_linear_acceleration> <!-- computed from <max_linear_acceleration> in the original plugin-->
-        <topic>cmd_vel</topic> <!-- from <commant_topic> -->
-        <odom_topic>odom</odom_topic> <!-- from <odometry_topic> -->
-        <frame_id>odom</frame_id> <!-- from <odometry_frame> -->
-        <child_frame_id>base_footprint</child_frame_id> <!-- from <robot_base_frame> -->
-        <odom_publisher_frequency>30</odom_publisher_frequency> <!-- from <update_rate>-->
-        <tf_topic>/tf</tf_topic> <!-- Short topic name for tf output -->
-      </plugin>
-      <!-- <plugin name="diff_drive_controller" filename="libgazebo_ros_diff_drive.so">
-        <legacyMode>false</legacyMode>
-        <alwaysOn>true</alwaysOn>
-        <updateRate>1000.0</updateRate>
-        <leftJoint>${left_wheel_joint}</leftJoint>
-        <rightJoint>${right_wheel_joint}</rightJoint>
-        <wheelSeparation>${wheel_separation}</wheelSeparation>
-        <wheelDiameter>${2*wheel_radius}</wheelDiameter>
-        <wheelTorque>10</wheelTorque>
-        <publishTf>1</publishTf>
-        <odometryFrame>map</odometryFrame>
-        <commandTopic>mobile_base_controller/cmd_vel</commandTopic>
-        <odometryTopic>mobile_base_controller/odom</odometryTopic>
-        <robotBaseFrame>base_footprint</robotBaseFrame>
-        <wheelAcceleration>2.8</wheelAcceleration>
-        <publishWheelJointState>true</publishWheelJointState>
-        <publishWheelTF>false</publishWheelTF>
-        <odometrySource>world</odometrySource>
-        <rosDebugLevel>Debug</rosDebugLevel>
-      </plugin> -->
-    </gazebo>
-  </xacro:macro>
   <xacro:macro name="set_wheel_friction" params="link friction">
     <gazebo reference="${link}">
@@ -60,17 +18,3 @@
     <xacro:set_wheel_friction link="${prefix}br_caster_wheel_link" friction="1"/>
   </xacro:macro>
-  <xacro:macro name="p3d_base_controller" params="prefix">
-    <!-- <gazebo>
-      <plugin name="p3d_base_controller" filename="libgazebo_ros_p3d.so">
-        <alwaysOn>true</alwaysOn>
-        <updateRate>50.0</updateRate>
-        <bodyName>${prefix}base_footprint</bodyName>
-        <topicName>base_pose_ground_truth</topicName>
-        <gaussianNoise>0.01</gaussianNoise>
-        <frameName>map</frameName>
-        <xyzOffsets>0 0 0</xyzOffsets>
-        <rpyOffsets>0 0 0</rpyOffsets>
-      </plugin>
-    </gazebo> -->
-  </xacro:macro>
 </robot>

File: mir/mir_description/urdf/include/mir_macro.xacro (robot description, xacro)
@@ -1,12 +1,9 @@
 <?xml version="1.0"?>
 <robot xmlns:xacro="http://ros.org/wiki/xacro">
-  <xacro:arg name="mir_type" default="mir_100" />   <!-- The MiR variant. Can be "mir_100" or "mir_250" for now.-->
+  <xacro:arg name="mir_type" default="mir_100" />   <!-- The MiR variant. Can be "mir_100" or "mir_200" for now.-->
   <xacro:property name="mir_type" value="$(arg mir_type)" />  <!-- necessary because args cannot be accessed inside ${} expressions -->
   <xacro:include filename="$(find mir_description)/urdf/include/common_properties.urdf.xacro" />
-  <xacro:include filename="$(find mir_description)/urdf/include/imu.gazebo.urdf.xacro" />
-  <xacro:include filename="$(find mir_description)/urdf/include/mir.gazebo.xacro" />
-  <xacro:include filename="$(find mir_description)/urdf/include/mir.transmission.xacro" />
   <xacro:include filename="$(find mir_description)/urdf/include/sick_s300.urdf.xacro" />
-  <xacro:property name="deg_to_rad" value="0.017453293" />
+  <xacro:property name="deg_to_rad" value="${pi/180}" />
   <!-- The inertia for the MiR platform is intentionally chosen to be smaller than
        the bounding box and also shifted a bit to the back, because most of the mass
@@ -135,10 +132,5 @@
         </geometry>
       </visual>
-      <!-- <collision>
-        <origin xyz="0 0 0" rpy="0 0 0" />
-        <geometry>
-          <mesh filename="package://mir_description/meshes/collision/caster_wheel_base.stl" />
-        </geometry>
-      </collision> -->
+      <!-- No collision mesh required -->
     </link>
     <!-- caster wheel -->
@@ -159,11 +151,4 @@
         </geometry>
       </visual>
-      <!-- <visual>
-        <origin xyz="0 0 0" rpy="${pi/2} 0 0" />
-        <geometry>
-          <cylinder radius="${mir_caster_wheel_radius}" length="${mir_caster_wheel_width}" />
-        </geometry>
-        <xacro:insert_block name="material_black" />
-      </visual> -->
       <collision>
         <origin xyz="0 0 0" rpy="${pi/2} 0 0" />
@@ -174,5 +159,5 @@
     </link>
   </xacro:macro>
-  <xacro:macro name="mir" params="prefix controller_config_file">
+  <xacro:macro name="mir" params="prefix">
     <link name="${prefix}base_footprint" />
     <joint name="${prefix}base_joint" type="fixed">
@@ -204,7 +189,5 @@
       <origin xyz="0.0 0.0 0.25" rpy="0 0 0" />  <!-- same as real MiR -->
     </joint>
-    <link name="${prefix}imu_link">
-      <xacro:imu_gazebo link="${prefix}imu_link" imu_topic="imu_data" update_rate="50.0" />
-    </link>
+    <link name="${prefix}imu_link" />
     <!-- Create an alias for imu_link. This is necessary because the real MiR's
          TF has imu_link, but the imu_data topic is published in the imu_frame
@@ -256,9 +239,4 @@
     </joint>
     <link name="${prefix}surface"/>
-    <xacro:mir_wheel_transmissions prefix="${prefix}"/>
-    <!-- set the gazebo friction parameters for the wheels -->
-    <xacro:set_all_wheel_frictions prefix="${prefix}"/>
-    <!-- <xacro:diff_controller_plugin_gazebo prefix="${prefix}" controller_config_file="${controller_config_file}" /> -->
-    <!-- <xacro:p3d_base_controller prefix="${prefix}" /> -->
   </xacro:macro>
 </robot>

File: mir/mir_description/urdf/include/sick_s300.urdf.xacro (robot description, xacro)
@@ -26,5 +26,5 @@
       </xacro:box_inertial>
     </link>
-    <gazebo reference="${prefix}${link}">
+    <!-- <gazebo reference="${prefix}${link}">
       <sensor name='${prefix}${link}' type='gpu_lidar'>
           <pose relative_to='${prefix}${link}'>0 0 0 0 0 0</pose>
@@ -56,5 +56,5 @@
           <visualize>true</visualize>
       </sensor>
-    </gazebo>
+    </gazebo> -->
   </xacro:macro>
 </robot>

File: mir/mir_description/urdf/mir.urdf (robot description, URDF)
Before this commit: robot mir, 19 links, 18 joints
Links:
- link imu_link: mass None -> 0.3097539019

File: mir/mir_description/urdf/mir.urdf.xacro (robot description, xacro)
@@ -1,8 +1,7 @@
 <?xml version="1.0"?>
-<robot xmlns:xacro="http://ros.org/wiki/xacro"
-       name="mir" >
-  <xacro:arg name="controller_config_file" default="$(find mir_description)/config/diff_drive_controller.yaml" />
+<robot name="mir" xmlns:xacro="http://www.ros.org/wiki/xacro">
   <!-- MiR base -->
-  <xacro:include filename="$(find mir_description)/urdf/include/mir_v2.urdf.xacro" />
+  <xacro:include filename="$(find mir_description)/urdf/include/mir_macro.xacro" />
+  <!-- Add common gazebo specific properties -->
   <xacro:include filename="$(find mir_description)/urdf/include/common.gazebo.xacro" />
   <xacro:arg name="tf_prefix" default="" />
@@ -14,13 +13,5 @@
     <xacro:property name="prefix" value="${tf_prefix_}/" />
   </xacro:unless>
-  <xacro:mir prefix="${prefix}" controller_config_file="$(arg controller_config_file)"/>
-  <xacro:arg name="simulation_engine" default="ignition-gazebo" />
-  <xacro:controller_plugin_gazebo robot_namespace=""/>
-  <!-- instead of the controller_plugin_gazebo, you can use the diffdrive controller like this
-    <xacro:diff_controller_plugin_gazebo prefix=""
-      left_wheel_joint="left_wheel_joint"
-      right_wheel_joint="right_wheel_joint"
-      wheel_separation="${2*mir_act_wheel_dy}"
-      wheel_radius="${mir_act_wheel_radius}"/>
-  -->
+  <xacro:mir prefix="${prefix}"/>
+  <xacro:gz_ros2 prefix="${prefix}"/>
 </robot>
