Commit message: created models for mir100 and mir200

File: mir/mir_description/urdf/include/common_properties.urdf.xacro (robot description, xacro)
@@ -50,4 +50,9 @@
     </material>
   </xacro:property>
+    <xacro:property name="material_blue">
+    <material name="silver">
+      <color rgba="0.1 0.1 0.8 1" />
+    </material>
+  </xacro:property>
   <!-- #################### inertials with origin #################### -->
   <!-- see https://secure.wikimedia.org/wikipedia/en/wiki/List_of_moment_of_inertia_tensors -->

File: mir/mir_description/urdf/include/imu.gazebo.urdf.xacro (robot description, xacro)
@@ -18,9 +18,9 @@
         <topicName>${imu_topic}</topicName>
         <accelDrift>0.0 0.0 0.0</accelDrift>
-        <accelGaussianNoise>${sqrt(5e-05)} ${sqrt(0.0001)} ${sqrt(0.00013)}</accelGaussianNoise>    <!-- real MiR linear_acceleration_covariance: [5e-05, 0.0, 0.0, 0.0, 0.0001, 0.0, 0.0, 0.0, 0.00013] -->
+        <accelGaussianNoise>${sqrt(5e-05)} ${sqrt(0.0001)} ${sqrt(0.00013)}</accelGaussianNoise>    <!-- real MiR linear_acceleration_covariance [5e-05, 0.0, 0.0, 0.0, 0.0001, 0.0, 0.0, 0.0, 0.00013] -->
         <rateDrift>0.0 0.0 0.0</rateDrift>
-        <rateGaussianNoise>${sqrt(8e-06)} ${sqrt(8e-06)} ${sqrt(3e-07)}</rateGaussianNoise>         <!-- real MiR angular_velocity_covariance: [8e-06, 0.0, 0.0, 0.0, 8e-06, 0.0, 0.0, 0.0, 3e-07] -->
+        <rateGaussianNoise>${sqrt(8e-06)} ${sqrt(8e-06)} ${sqrt(3e-07)}</rateGaussianNoise>         <!-- real MiR angular_velocity_covariance [8e-06, 0.0, 0.0, 0.0, 8e-06, 0.0, 0.0, 0.0, 3e-07] -->
         <yawDrift>0.0</yawDrift>
-        <yawGaussianNoise>${sqrt(0.1)}</yawGaussianNoise>                                           <!-- real MiR orientation_covariance: [0.1, 0.0, 0.0, 0.0, 0.1, 0.0, 0.0, 0.0, 0.1] -->
+        <yawGaussianNoise>${sqrt(0.1)}</yawGaussianNoise>                                           <!-- real MiR orientation_covariance [0.1, 0.0, 0.0, 0.0, 0.1, 0.0, 0.0, 0.0, 0.1] -->
       </plugin>
     </gazebo>

File: mir/mir_description/urdf/include/mir_v1.urdf.xacro (robot description, xacro)
@@ -1,5 +1,5 @@
 <?xml version="1.0"?>
 <robot xmlns:xacro="http://ros.org/wiki/xacro">
-  <xacro:arg name="mir_type" default="mir_100" />      <!-- The MiR variant. Can be "mir_100" or "mir_250" for now.-->
+  <xacro:arg name="mir_type" default="mir_100" />   <!-- The MiR variant. Can be "mir_100" or "mir_250" for now.-->
   <xacro:property name="mir_type" value="$(arg mir_type)" />  <!-- necessary because args cannot be accessed inside ${} expressions -->
   <xacro:include filename="$(find mir_description)/urdf/include/common_properties.urdf.xacro" />
@@ -19,5 +19,13 @@
   <xacro:property name="mir_base_inertial_z_length" value="0.20" />
   <xacro:if value="${mir_type == 'mir_100'}">
-    <xacro:property name="mir_base_mass" value="77.0" />
+    <xacro:property name="mir_base_mass" value="62.5" />
+    <xacro:property name="mir_act_wheel_radius" value="0.0625" />
+    <xacro:property name="mir_act_wheel_width" value="0.032" />
+    <xacro:property name="mir_act_wheel_mass" value="1.0" />
+    <xacro:property name="mir_act_wheel_dx" value="0.037646" />
+    <xacro:property name="mir_act_wheel_dy" value="0.222604" />
+  </xacro:if>
+  <xacro:if value="${mir_type == 'mir_200'}">
+    <xacro:property name="mir_base_mass" value="70.0" />
     <xacro:property name="mir_act_wheel_radius" value="0.0625" />
     <xacro:property name="mir_act_wheel_width" value="0.032" />
@@ -45,4 +53,8 @@
     <xacro:property name="mir_caster_wheel_base_dy" value="0.203" />
   </xacro:if>
+  <xacro:if value="${mir_type == 'mir_200'}">
+    <xacro:property name="mir_back_caster_wheel_base_dx"  value="0.3078" />
+    <xacro:property name="mir_caster_wheel_base_dy" value="0.203" />
+  </xacro:if>
   <xacro:if value="${mir_type == 'mir_250'}">
     <xacro:property name="mir_back_caster_wheel_base_dx"  value="0.296" />
@@ -55,4 +67,8 @@
     <xacro:property name="laser_dy" value="0.2358" />
   </xacro:if>
+  <xacro:if value="${mir_type == 'mir_200'}">
+    <xacro:property name="laser_dx" value="0.392" />
+    <xacro:property name="laser_dy" value="0.2358" />
+  </xacro:if>
   <xacro:if value="${mir_type == 'mir_250'}">
     <xacro:property name="laser_dx" value="0.315" />
@@ -87,5 +103,5 @@
     </link>
     <gazebo reference="${prefix}${locationprefix}_wheel_link">
-      <material>Gazebo/FlatBlack</material>
+      <material>Gazebo/Blue</material>
     </gazebo>
   </xacro:macro>
@@ -202,4 +218,7 @@
         <material>Gazebo/White</material>
       </xacro:if>
+      <xacro:if value="${mir_type == 'mir_200'}">
+        <material>Gazebo/Grey</material>
+      </xacro:if>
       <xacro:if value="${mir_type == 'mir_250'}">
         <material>Gazebo/DarkGrey</material>

File: mir/mir_description/urdf/include/sick_s300.urdf.xacro (robot description, xacro)
@@ -9,17 +9,17 @@
     <link name="${prefix}${link}">
       <visual>
+        <origin xyz="-0.335 -0.385 0.1555" rpy="0 0 ${3*pi/4}" />
+        <geometry>
+          <mesh filename="package://mir_description/meshes/mir_100/visual/SICK-lidar.dae" />
+        </geometry>
+        <!-- <xacro:insert_block name="material_yellow" /> -->
+        <!-- <xacro:insert_block name="material_black" /> -->
+      </visual>
+      <!-- <collision>
         <origin xyz="0.0 0.0 0.0" rpy="${pi} 0 0" />
         <geometry>
-          <mesh filename="package://mir_description/meshes/visual/sick_lms-100.stl" />
+          <mesh filename="package://mir_description/meshes/mir_100/visual/SICK-lidar.dae" />
         </geometry>
-        <!-- <xacro:insert_block name="material_yellow" /> -->
-        <xacro:insert_block name="material_black" />
-      </visual>
-      <collision>
-        <origin xyz="0.0 0.0 0.0" rpy="${pi} 0 0" />
-        <geometry>
-          <mesh filename="package://mir_description/meshes/visual/sick_lms-100.stl" />
-        </geometry>
-      </collision>
+      </collision> -->
       <xacro:box_inertial x="${laser_x}" y="${laser_y}" z="${laser_z}" mass="${laser_mass}">
         <origin xyz="0 0 0" />
@@ -28,5 +28,5 @@
     <gazebo reference="${prefix}${link}">
       <!-- <material value="Gazebo/Yellow" /> -->
-      <material value="Gazebo/FlatBlack" />
+      <!-- <material value="Gazebo/FlatBlack" /> -->
       <sensor type="ray" name="${prefix}${link}">
         <pose>0 0 0 0 0 0</pose>

File: mir/mir_description/urdf/mir.urdf.xacro (robot description, xacro)
@@ -3,5 +3,5 @@
        name="mir" >
   <!-- MiR base -->
-  <xacro:include filename="$(find mir_description)/urdf/include/mir_v1.urdf.xacro" />
+  <xacro:include filename="$(find mir_description)/urdf/include/mir_v2.urdf.xacro" />
   <xacro:include filename="$(find mir_description)/urdf/include/common.gazebo.xacro" />
   <xacro:arg name="tf_prefix" default="" />
@@ -15,5 +15,5 @@
   <xacro:mir prefix="${prefix}" />
   <xacro:controller_plugin_gazebo robot_namespace=""/>
-  <!-- instead of the controller_plugin_gazebo, you can use the diffdrive controller like this:
+  <!-- instead of the controller_plugin_gazebo, you can use the diffdrive controller like this
     <xacro:diff_controller_plugin_gazebo prefix=""
       left_wheel_joint="left_wheel_joint"

Commit message: separated gazebo package

File: mir/mir_description/urdf/include/common_properties.urdf.xacro (robot description, xacro)
@@ -40,9 +40,9 @@
     </material>
   </xacro:property>
-  <xacro:property name="material_aluminum">
+  <!-- <xacro:property name="material_aluminum">
     <material name="aluminum">
       <color rgba="0.8 0.8 0.8 1" />
     </material>
-  </xacro:property>
+  </xacro:property> -->
   <xacro:property name="material_silver">
     <material name="silver">

File: mir/mir_description/urdf/include/mir_macro.xacro (robot description, xacro)
@@ -3,6 +3,9 @@
   <xacro:arg name="mir_type" default="mir_100" />   <!-- The MiR variant. Can be "mir_100" or "mir_200" for now.-->
   <xacro:property name="mir_type" value="$(arg mir_type)" />  <!-- necessary because args cannot be accessed inside ${} expressions -->
+  <xacro:arg name="use_nominal_extrinsics" default="false" />
+  <xacro:property name="use_nominal_extrinsics" value="$(arg use_nominal_extrinsics)" />
   <xacro:include filename="$(find mir_description)/urdf/include/common_properties.urdf.xacro" />
   <xacro:include filename="$(find mir_description)/urdf/include/sick_s300.urdf.xacro" />
+  <xacro:include filename="$(find mir_description)/urdf/include/realsense_camera.urdf.xacro" />
   <xacro:property name="deg_to_rad" value="${pi/180}" />
   <!-- The inertia for the MiR platform is intentionally chosen to be smaller than
@@ -73,4 +76,17 @@
   </xacro:if>
   <xacro:property name="laser_dz" value="0.1914" />
+  <!-- from visually matching up the meshes of the MiR and the 3D cameras -->
+  <xacro:if value="${mir_type == 'mir_100'}">
+    <xacro:property name="camera_dx" value="-0.025" />
+    <xacro:property name="camera_dy" value="0.08125" />
+  </xacro:if>
+  <xacro:if value="${mir_type == 'mir_200'}">
+    <xacro:property name="camera_dx" value="-0.025" />
+    <xacro:property name="camera_dy" value="0.08125" />
+  </xacro:if>
+  <!-- TODO: Find the values of the camera dx and dy -->
+  <xacro:if value="${mir_type == 'mir_250'}">
+  </xacro:if>
+  <xacro:property name="camera_dz" value="-0.015" />
   <xacro:macro name="actuated_wheel" params="prefix locationprefix locationright">
     <joint name="${prefix}${locationprefix}_wheel_joint" type="continuous">
@@ -159,5 +175,5 @@
     </link>
   </xacro:macro>
-  <xacro:macro name="mir" params="prefix">
+  <xacro:macro name="mir" params="prefix use_nominal_extrinsics">
     <link name="${prefix}base_footprint" />
     <joint name="${prefix}base_joint" type="fixed">
@@ -212,4 +228,28 @@
     </joint>
     <xacro:sick_s300 prefix="${prefix}" link="back_laser_link" topic="b_scan" />
+    <!-- 3D cameras -->
+    <!-- Charging point -->
+    <link name="${prefix}charge_point_link" />
+    <joint name="${prefix}base_link_to_charging_link" type="fixed">
+      <parent link="${prefix}base_link" />
+      <child link="${prefix}charge_point_link" />
+      <origin xyz="0.4675 0.0 0.13" rpy="0.0 0.0 0.0" />
+    </joint>
+    <joint name="${prefix}charge_point_link_to_camera1" type="fixed">
+      <parent link="${prefix}charge_point_link" />
+      <child link="${prefix}camera_1_link" />
+      <origin xyz="${camera_dx} ${camera_dy} ${camera_dz}" rpy="${-pi/2} -0.37 ${-pi/3}" />
+    </joint>
+    <xacro:realsense_cameras prefix="${prefix}" link="camera_1_link" name="camera1" use_nominal_extrinsics="${use_nominal_extrinsics}" add_plug="false" use_mesh="true">
+      <origin xyz="0.01 0.001 -0.02" rpy="0 ${-pi/6} 0"/>
+    </xacro:realsense_cameras>
+    <joint name="${prefix}charge_point_link_to_camera2" type="fixed">
+      <parent link="${prefix}charge_point_link" />
+      <child link="${prefix}camera_2_link" />
+      <origin xyz="${camera_dx} -${camera_dy} ${camera_dz}" rpy="${-pi/2} -0.35 ${pi/3}" />
+    </joint>
+    <xacro:realsense_cameras prefix="${prefix}" link="camera_2_link" name="camera2" use_nominal_extrinsics="${use_nominal_extrinsics}" add_plug="false" use_mesh="true">
+      <origin xyz="0 0 0" rpy="0 ${pi/6} 0"/>
+    </xacro:realsense_cameras>
     <!-- Ultrasound sensors -->
     <joint name="${prefix}us_1_joint" type="fixed">   <!-- right ultrasound -->

File: mir/mir_description/urdf/include/sick_s300.urdf.xacro (robot description, xacro)
@@ -13,7 +13,6 @@
           <mesh filename="package://mir_description/meshes/mir_100/visual/SICK-lidar.dae" />
         </geometry>
-        <!-- <xacro:insert_block name="material_yellow" /> -->
-        <!-- <xacro:insert_block name="material_black" /> -->
       </visual>
+      <!-- Collision model is not necessary -->
       <!-- <collision>
         <origin xyz="0.0 0.0 0.0" rpy="${pi} 0 0" />
@@ -26,35 +25,4 @@
       </xacro:box_inertial>
     </link>
-    <!-- <gazebo reference="${prefix}${link}">
-      <sensor name='${prefix}${link}' type='gpu_lidar'>
-          <pose relative_to='${prefix}${link}'>0 0 0 0 0 0</pose>
-          <topic>${topic}</topic>
-          <update_rate>12.5</update_rate>
-          <gz_frame_id>base_scan</gz_frame_id>
-          <lidar>
-              <scan>
-                  <horizontal>
-                      <samples>541</samples>
-                      <resolution>1</resolution>
-                      <min_angle>-2.35619449615</min_angle>
-                      <max_angle>2.35619449615</max_angle>
-                  </horizontal>
-                  <vertical>
-                      <samples>1</samples>
-                      <resolution>0.01</resolution>
-                      <min_angle>0</min_angle>
-                      <max_angle>0</max_angle>
-                  </vertical>
-              </scan>
-              <range>
-                  <min>0.05</min>
-                  <max>29.0</max>
-                  <resolution>0.01</resolution>
-              </range>
-          </lidar>
-          <always_on>true</always_on>
-          <visualize>true</visualize>
-      </sensor>
-    </gazebo> -->
   </xacro:macro>
 </robot>

File: mir/mir_gazebo/urdf/mir.urdf (robot description, URDF)
Before this commit: robot mir, 25 links, 24 joints
Links:
- added link charge_point_link
Joints:
- removed joint base_link_to_camera1
- removed joint base_link_to_camera2
- added joint base_link_to_charging_link: type fixed, parent base_link, child charge_point_link, origin xyz=0.4675 0.0 0.13 rpy=0.0 0.0 0.0
- added joint charge_point_link_to_camera1: type fixed, parent charge_point_link, child camera_1_link, origin xyz=-0.025 0.08125 -0.015 rpy=-1.5707963267948966 -0.37 -1.0471975511965976
- added joint charge_point_link_to_camera2: type fixed, parent charge_point_link, child camera_2_link, origin xyz=-0.025 -0.08125 -0.015 rpy=-1.5707963267948966 -0.35 1.0471975511965976
- joint camera1_joint: origin xyz=0 0 0 rpy=0 0 0 -> xyz=0.01 0.001 -0.02 rpy=0 -0.5235987755982988 0
- joint camera2_joint: origin xyz=0 0 0 rpy=0 0 0 -> xyz=0 0 0 rpy=0 0.5235987755982988 0

File: mir/mir_gazebo/urdf/mir.urdf.xacro (robot description, xacro)
@@ -3,4 +3,6 @@
   <!-- MiR base -->
   <xacro:include filename="$(find mir_description)/urdf/include/mir_macro.xacro" />
+  <!-- Add common gazebo specific properties -->
+  <xacro:include filename="$(find mir_gazebo)/urdf/include/macro.gazebo.xacro" />
   <xacro:arg name="tf_prefix" default="" />
   <xacro:property name="tf_prefix_" value="$(arg tf_prefix)" />
@@ -15,3 +17,4 @@
   <xacro:property name="use_nominal_extrinsics" value="$(arg use_nominal_extrinsics)" />
   <xacro:mir prefix="${prefix}" use_nominal_extrinsics="${use_nominal_extrinsics}" />
+  <xacro:gz_ros2 prefix="${prefix}"/>
 </robot>
