Commit message: added realsense2 camera

File: mir/mir_description/urdf/include/mir_macro.xacro (robot description, xacro)
@@ -228,5 +228,4 @@
     </joint>
     <xacro:sick_s300 prefix="${prefix}" link="back_laser_link" topic="b_scan" />
-    <!-- 3D cameras -->
     <!-- Charging point -->
     <link name="${prefix}charge_point_link" />
@@ -236,4 +235,5 @@
       <origin xyz="0.4675 0.0 0.13" rpy="0.0 0.0 0.0" />
     </joint>
+    <!-- 3D cameras -->
     <joint name="${prefix}charge_point_link_to_camera1" type="fixed">
       <parent link="${prefix}charge_point_link" />

File: mir/mir_gazebo/urdf/include/imu.gazebo.xacro (robot description, xacro)
@@ -20,5 +20,4 @@
                             <dynamic_bias_stddev>0.00002</dynamic_bias_stddev>
                             <dynamic_bias_correlation_time>400.0</dynamic_bias_correlation_time>
-                            <precision>0.00025</precision>
                         </noise>
                         </x>
@@ -31,5 +30,4 @@
                             <dynamic_bias_stddev>0.00002</dynamic_bias_stddev>
                             <dynamic_bias_correlation_time>400.0</dynamic_bias_correlation_time>
-                            <precision>0.00025</precision>
                         </noise>
                         </y>
@@ -42,5 +40,4 @@
                             <dynamic_bias_stddev>0.00002</dynamic_bias_stddev>
                             <dynamic_bias_correlation_time>400.0</dynamic_bias_correlation_time>
-                            <precision>0.00025</precision>
                         </noise>
                         </z>
@@ -55,5 +52,4 @@
                             <dynamic_bias_stddev>0.000375</dynamic_bias_stddev>
                             <dynamic_bias_correlation_time>175.0</dynamic_bias_correlation_time>
-                            <precision>0.005</precision>
                         </noise>
                         </x>
@@ -66,5 +62,4 @@
                             <dynamic_bias_stddev>0.000375</dynamic_bias_stddev>
                             <dynamic_bias_correlation_time>175.0</dynamic_bias_correlation_time>
-                            <precision>0.005</precision>
                         </noise>
                         </y>
@@ -77,5 +72,4 @@
                             <dynamic_bias_stddev>0.000375</dynamic_bias_stddev>
                             <dynamic_bias_correlation_time>175.0</dynamic_bias_correlation_time>
-                            <precision>0.005</precision>
                         </noise>
                         </z>

File: mir/mir_gazebo/urdf/include/macro.gazebo.xacro (robot description, xacro)
@@ -3,5 +3,6 @@
     <xacro:include filename="$(find mir_gazebo)/urdf/include/control.gazebo.xacro" />
     <xacro:include filename="$(find mir_gazebo)/urdf/include/imu.gazebo.xacro" />
-    <xacro:include filename="$(find mir_gazebo)/urdf/include/lidar.gazebo.xacro" />
+    <xacro:include filename="$(find mir_gazebo)/urdf/include/scanner.gazebo.xacro" />
+    <xacro:include filename="$(find mir_gazebo)/urdf/include/depthcamera.gazebo.xacro" />
     <xacro:macro name="gz_ros2" params="prefix">
       <xacro:gz_ros2_control prefix="${prefix}" />
@@ -18,4 +19,5 @@
         <plugin
           filename="gz-sim-sensors-system" name="gz::sim::systems::Sensors">
+          <frame_id>custom_params/link</frame_id>
           <render_engine>ogre2</render_engine>
         </plugin>
@@ -26,5 +28,8 @@
       </gazebo>
       <xacro:imu_gazebo prefix="${prefix}" />
-      <xacro:lidar_gazebo prefix="${prefix}" />
+      <xacro:scanner_gazebo prefix="${prefix}" location="front" />
+      <xacro:scanner_gazebo prefix="${prefix}" location="back" />
+      <xacro:realsense2_gazebo prefix="${prefix}" camera_name="camera1" />
+      <xacro:realsense2_gazebo prefix="${prefix}" camera_name="camera2" />
     </xacro:macro>
 </robot>

File: mir/mir_gazebo/urdf/mir.urdf (robot description, URDF)
Before this commit: robot mir, 26 links, 25 joints
Links:
- added link back_laser_frame
- added link front_laser_frame
Joints:
- added joint back_laser_link_to_back_laser_frame_joint: type fixed, parent back_laser_link, child back_laser_frame, origin xyz=0 0 0 rpy=0 0 0
- added joint front_laser_link_to_front_laser_frame_joint: type fixed, parent front_laser_link, child front_laser_frame, origin xyz=0 0 0 rpy=0 0 0
