Commit message: commit after long time

File: mir/mir_gazebo/urdf/include/depthcamera.gazebo.xacro (robot description, xacro)
@@ -3,5 +3,5 @@
 <!-- Realsense2 camera in gazebo - https://github.com/pal-robotics/realsense_simulation/ -->
 <robot xmlns:xacro="http://ros.org/wiki/xacro">
-  <xacro:macro name="realsense2_gazebo" params="prefix camera_name">
+  <xacro:macro name="realsense2_gazebo" params="prefix camera_name update_rate">
     <gazebo reference="${camera_name}_link">
       <self_collide>0</self_collide>
@@ -25,6 +25,6 @@
           <camera_info_topic>${camera_name}/color/image/info</camera_info_topic>
           <image>
-            <width>640</width>
-            <height>480</height>
+            <width>424</width>
+            <height>240</height>
             <format>RGB_INT8</format>
           </image>
@@ -43,5 +43,5 @@
         </camera>
         <always_on>1</always_on>
-        <update_rate>30</update_rate>
+        <update_rate>${update_rate}</update_rate>
         <visualize>1</visualize>
       </sensor>
@@ -53,6 +53,6 @@
           <camera_info_topic>${camera_name}/infra1/image/info</camera_info_topic>
           <image>
-            <width>1280</width>
-            <height>720</height>
+            <width>640</width>
+            <height>480</height>
             <format>L8</format>
           </image>
@@ -68,5 +68,5 @@
         </camera>
         <always_on>1</always_on>
-        <update_rate>30</update_rate>
+        <update_rate>${update_rate}</update_rate>
         <visualize>0</visualize>
       </sensor>
@@ -78,6 +78,6 @@
           <camera_info_topic>${camera_name}/infra2/image/info</camera_info_topic>
           <image>
-            <width>1280</width>
-            <height>720</height>
+            <width>640</width>
+            <height>480</height>
             <format>L8</format>
           </image>
@@ -93,5 +93,5 @@
         </camera>
         <always_on>1</always_on>
-        <update_rate>30</update_rate>
+        <update_rate>${update_rate}</update_rate>
         <visualize>0</visualize>
       </sensor>
@@ -102,6 +102,6 @@
           <horizontal_fov>${85.2*pi/180}</horizontal_fov>
           <image>
-            <width>1280</width>
-            <height>720</height>
+            <width>320</width>
+            <height>240</height>
           </image>
           <clip>
@@ -123,5 +123,5 @@
         </camera>
         <always_on>1</always_on>
-        <update_rate>30</update_rate>
+        <update_rate>${update_rate}</update_rate>
         <visualize>0</visualize>
       </sensor>

File: mir/mir_gazebo/urdf/include/macro.gazebo.xacro (robot description, xacro)
@@ -30,6 +30,6 @@
       <xacro:scanner_gazebo prefix="${prefix}" location="front" />
       <xacro:scanner_gazebo prefix="${prefix}" location="back" />
-      <xacro:realsense2_gazebo prefix="${prefix}" camera_name="camera1" />
-      <xacro:realsense2_gazebo prefix="${prefix}" camera_name="camera2" />
+      <xacro:realsense2_gazebo prefix="${prefix}" camera_name="camera1" update_rate="1" />
+      <xacro:realsense2_gazebo prefix="${prefix}" camera_name="camera2" update_rate="1" />
     </xacro:macro>
 </robot>
